Commit message: fix a few joint

File: ForteME.urdf (robot description, URDF)
Before this commit: robot ForteME_urdf, 7 links, 6 joints
Links:
- removed link shoulder_roll_link
- added link lower_arm_link, mass 0.53088093; collision mesh filename=package://meshes/lower_arm_link.stl; visual mesh filename=package://meshes/lower_arm_link.stl
- added link shoulder_pitch_link, mass 0.59865534; collision mesh filename=package://meshes/shoulder_pitch_link.stl; visual mesh filename=package://meshes/shoulder_pitch_link.stl
- link elbow_link: mass 0.91715589 -> 0.38627496
Joints:
- added joint lower_arm_roll: type revolute, parent elbow_link, child lower_arm_link, origin xyz=0.06050000 0.03400000 0.03500000 rpy=0 0 0, axis 1 0 0, limit lower=-3.141592653589793 upper=3.141592653589793 effort=10 velocity=10
- joint shoulder_pitch: axis 1 0 0 -> 0 1 0; child upper_arm_link -> shoulder_pitch_link; origin xyz=0.00050000 0.06300000 0 rpy=0 0 0 -> xyz=0 -0.06300000 0.12500000 rpy=0 0 0; parent shoulder_roll_link -> shoulder_yaw_link
- joint shoulder_roll: axis 0 1 0 -> 1 0 0; child shoulder_roll_link -> upper_arm_link; origin xyz=0 -0.06300000 0.12500000 rpy=0 0 0 -> xyz=0.00050000 0.06300000 0 rpy=0 0 0; parent shoulder_yaw_link -> shoulder_pitch_link
- joint wrist_pitch: origin xyz=0.44700000 0.00550000 0.03500000 rpy=0 0 0 -> xyz=0.38650000 -0.02850000 0 rpy=0 0 0; parent elbow_link -> lower_arm_link
